File: hardware/servo.kicad_sch (KiCad schematic)
At the start: 37 parts, among them J1 servo, J2 Jack-DC, J3 swd, Q2 DMT64M8LSS, SW1 restart, SW2 buzzer, U1 AOZ1284PI, U3 STM32G030F6Px, U4 LDI1117-3.3U-DIO

Commit message: fix barrel jack footprint
Parts:
- J2: footprint Connector_BarrelJack:BarrelJack_CUI_PJ-102AH_Horizontal -> Connector_BarrelJack:BarrelJack_diy
Changed lines of the file:
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@@
 			)
 		)
-		(property "Footprint" "Connector_BarrelJack:BarrelJack_CUI_PJ-102AH_Horizontal"
+		(property "Footprint" "Connector_BarrelJack:BarrelJack_diy"
 			(at 26.67 31.496 0)
 			(hide yes)

Commit message: schematic cleanup, repo organizing
Other:
- note removed: "FT pin"
- moved on the sheet: BZ1, C1, C10, C2, C3, C4, C5, C6, C7, C8, C9, D1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
