File: hardware/servo.kicad_sch (KiCad schematic)
At the start: 37 parts, among them J1 servo, J2 Jack-DC, J3 swd, Q2 DMT64M8LSS, SW1 restart, SW2 buzzer, U1 AOZ1284PI, U3 STM32G030F6Px, U4 LDI1117-3.3U-DIO

Commit message: Fix getting stuck in bootloader, false overcurrent triggers
HARDWARE: add BOOT0 pulldown, reduce buzzer resistance for more volume, add drill hole for AOZ1284 footprint EPAD
SOFTWARE: add ADC delay for motor inrush, add software lowpass filtering to overcurrent protection
Parts:
- added R10: 10k, Resistor_SMD:R_0805_2012Metric_Pad1.20x1.40mm_HandSolder, symbol Device:R
- R7: value 51k -> 300
- U1: footprint Package_SO:SOIC-8-1EP_3.9x4.9mm_P1.27mm_EP2.71x3.7mm -> Package_SO:SOIC-8-1EP_3.9x4.9mm_P1.27mm_EP2.29x3mm_diy
Connections:
- net GND: now also R10.2
- net swclk: now also R10.1
Other:
- moved on the sheet: D1, D3, J1, Q2, R5, R6

Commit message: Hardware and software fixes, reorganize
Recalculate compensation for 4.7mF, increase ADC delay, improve code readability, match compensation annotation in schematic to datasheet
Parts:
- added Cc1: 150p, Capacitor_SMD:C_0805_2012Metric_Pad1.18x1.45mm_HandSolder, symbol Device:C
- Cc2: renamed from C6; value 1.5n -> 6.8n
- Rc1: renamed from R4; value 10k -> 1M
- renumbered C2 to C1, C10 to C2, C1 to C3, C5 to C4, C3 to C5, C9 to C6, C4 to C7, C7 to C8, C8 to C9, J2 to J1, J1 to J2, Q2 to Q1, R8 to R1, R9 to R2, R1 to R3, R2 to R4, R3 to R5, R5 to R6, R6 to R7, R10 to R8, R7 to R9, U4 to U2
Connections:
- net GND: now also Cc1.2
- net at Rc1.1, U1.5 (COMP): now also Cc1.1
Other:
- moved on the sheet: C1, C3, C5, C7, Cc2, D2, L1, R1, R2, R3, R4, R5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
